File: schematics/project/ice_wheel.kicad_pcb (KiCad board)
At the start: 2 copper layers, 2 parts, among them U1 OPA320xxDBV, U2 Teensy4.1

Commit message: Structure of schematics
Parts:
- added C1: C, Capacitor_SMD:C_0603_1608Metric, F.Cu at (124.5, 88.9)
- added C2: 100nF 10V, Capacitor_SMD:C_0603_1608Metric, F.Cu at (128.5, 91.4)
- added R1: R, Resistor_SMD:R_0603_1608Metric, F.Cu at (128.5, 88.9)
- added R2: R, Resistor_SMD:R_0603_1608Metric, F.Cu at (124.5, 93.9)
- added R3: R, Resistor_SMD:R_0603_1608Metric, F.Cu at (124.5, 91.4)
Connections:
- U1 pad 1: unconnected-(U1-Pad1) -> /SetSpeed_Analog
- U1 pad 2: unconnected-(U1-Pad2) -> GND
- U1 pad 3: unconnected-(U1-Pad3) -> Net-(U1-Pad3)
- U1 pad 4: unconnected-(U1-Pad4) -> Net-(U1-Pad4)
- U1 pad 5: unconnected-(U1-Pad5) -> +5V
