File: schematics/project/3speed.kicad_sch (KiCad schematic)
At the start: 2 parts

Commit message: First steps with kicad structure -> kinda sucks
Parts:
- gave numbers to parts that had none: 2
Changed lines of the file:
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@@
   (symbol (lib_id "Device:R") (at 111.76 81.28 270) (unit 1)
     (in_bom yes) (on_board yes) (fields_autoplaced)
-    (property "Reference" "R?" (id 0) (at 111.76 74.93 90))
+    (property "Reference" "R4" (id 0) (at 111.76 74.93 90))
     (property "Value" "1k" (id 1) (at 111.76 77.47 90))
     (property "Footprint" "Resistor_SMD:R_0603_1608Metric" (id 2) (at 111.76 79.502 90)
@@
   (symbol (lib_id "power:GND") (at 128.27 91.44 0) (unit 1)
     (in_bom yes) (on_board yes) (fields_autoplaced)
-    (property "Reference" "#PWR?" (id 0) (at 128.27 97.79 0)
+    (property "Reference" "#PWR0109" (id 0) (at 128.27 97.79 0)
       (effects (font (size 1.27 1.27)) hide)
     )
@@
   (symbol (lib_id "Transistor_FET:BSS123") (at 125.73 81.28 0) (unit 1)
     (in_bom yes) (on_board yes) (fields_autoplaced)
-    (property "Reference" "Q?" (id 0) (at 132.08 80.0099 0)
+    (property "Reference" "Q1" (id 0) (at 132.08 80.0099 0)
       (effects (font (size 1.27 1.27)) (justify left))
     )
