File: schematics/project/_autosave-ice_wheel.kicad_pcb (KiCad board)
At the start: 2 copper layers, 16 parts, among them Q1 BSS123, U1 OPA320xxDBV, U1 Teensy4.1, U2 PropShieldMotionSens, U3 OPA320xxDBV

Commit message: First steps with kicad structure -> kinda sucks
Connections:
- U1 pad 12: /Teensy/CS -> /Prop Shield/CS
- U1 pad 13: /Teensy/MOSI -> /Prop Shield/MOSI
- U1 pad 14: /Teensy/MISO -> /Prop Shield/MISO
- U1 pad 35: /Teensy/SCK -> /Prop Shield/SCK
- U1 pad 4: /Teensy/IRQ -> /Prop Shield/IRQ
- U1 pad 40: /Teensy/SDA -> /Prop Shield/SDA
- U1 pad 41: /Teensy/SCL -> /Prop Shield/SCL
