File: schematics/project/dig2anal.kicad_sch (KiCad schematic)
At the start: 6 parts

Commit message: First steps with kicad structure -> kinda sucks
Parts:
- gave numbers to parts that had none: 6
Changed lines of the file:
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@@
   (symbol (lib_id "power:GND") (at 158.75 92.71 0) (unit 1)
     (in_bom yes) (on_board yes) (fields_autoplaced)
-    (property "Reference" "#PWR?" (id 0) (at 158.75 99.06 0)
+    (property "Reference" "#PWR0104" (id 0) (at 158.75 99.06 0)
       (effects (font (size 1.27 1.27)) hide)
     )
@@
   (symbol (lib_id "Device:R") (at 143.51 86.36 90) (unit 1)
     (in_bom yes) (on_board yes)
-    (property "Reference" "R?" (id 0) (at 142.24 83.82 90))
+    (property "Reference" "R2" (id 0) (at 142.24 83.82 90))
     (property "Value" "R" (id 1) (at 142.24 88.9 90))
     (property "Footprint" "Resistor_SMD:R_0603_1608Metric" (id 2) (at 143.51 88.138 90)
@@
   (symbol (lib_id "power:GND") (at 133.35 96.52 0) (unit 1)
     (in_bom yes) (on_board yes) (fields_autoplaced)
-    (property "Reference" "#PWR?" (id 0) (at 133.35 102.87 0)
+    (property "Reference" "#PWR0105" (id 0) (at 133.35 102.87 0)
       (effects (font (size 1.27 1.27)) hide)
     )
@@
   (symbol (lib_id "Amplifier_Operational:OPA330xxDBV") (at 161.29 83.82 0) (unit 1)
     (in_bom yes) (on_board yes) (fields_autoplaced)
-    (property "Reference" "U?" (id 0) (at 173.99 79.121 0))
+    (property "Reference" "U3" (id 0) (at 173.99 79.121 0))
     (property "Value" "OPA320xxDBV" (id 1) (at 173.99 81.661 0))
     (property "Footprint" "Package_TO_SOT_SMD:SOT-23-5" (id 2) (at 158.75 88.9 0)
@@
   (symbol (lib_id "Device:C") (at 129.54 88.9 0) (unit 1)
     (in_bom yes) (on_board yes) (fields_autoplaced)
-    (property "Reference" "C?" (id 0) (at 133.35 87.6299 0)
+    (property "Reference" "C1" (id 0) (at 133.35 87.6299 0)
       (effects (font (size 1.27 1.27)) (justify left))
     )
@@
   (symbol (lib_id "power:GND") (at 167.64 76.2 0) (unit 1)
     (in_bom yes) (on_board yes) (fields_autoplaced)
-    (property "Reference" "#PWR?" (id 0) (at 167.64 82.55 0)
+    (property "Reference" "#PWR0107" (id 0) (at 167.64 82.55 0)
       (effects (font (size 1.27 1.27)) hide)
     )
@@
   (symbol (lib_id "power:+5V") (at 158.75 74.93 0) (unit 1)
     (in_bom yes) (on_board yes) (fields_autoplaced)
-    (property "Reference" "#PWR?" (id 0) (at 158.75 78.74 0)
+    (property "Reference" "#PWR0106" (id 0) (at 158.75 78.74 0)
       (effects (font (size 1.27 1.27)) hide)
     )
@@
   (symbol (lib_id "Device:R") (at 149.86 95.25 180) (unit 1)
     (in_bom yes) (on_board yes) (fields_autoplaced)
-    (property "Reference" "R?" (id 0) (at 152.4 93.9799 0)
+    (property "Reference" "R3" (id 0) (at 152.4 93.9799 0)
       (effects (font (size 1.27 1.27)) (justify right))
     )
@@
   (symbol (lib_id "power:+5V") (at 167.64 66.04 0) (unit 1)
     (in_bom yes) (on_board yes) (fields_autoplaced)
-    (property "Reference" "#PWR?" (id 0) (at 167.64 69.85 0)
+    (property "Reference" "#PWR0108" (id 0) (at 167.64 69.85 0)
       (effects (font (size 1.27 1.27)) hide)
     )
@@
   (symbol (lib_id "Device:C") (at 167.64 71.12 0) (unit 1)
     (in_bom yes) (on_board yes) (fields_autoplaced)
-    (property "Reference" "C?" (id 0) (at 171.45 69.8499 0)
+    (property "Reference" "C2" (id 0) (at 171.45 69.8499 0)
       (effects (font (size 1.27 1.27)) (justify left))
     )
@@
   (symbol (lib_id "Device:R") (at 121.92 81.28 90) (unit 1)
     (in_bom yes) (on_board yes) (fields_autoplaced)
-    (property "Reference" "R?" (id 0) (at 121.92 74.93 90))
+    (property "Reference" "R1" (id 0) (at 121.92 74.93 90))
     (property "Value" "R" (id 1) (at 121.92 77.47 90))
     (property "Footprint" "Resistor_SMD:R_0603_1608Metric" (id 2) (at 121.92 83.058 90)

Commit message: some progress, dust slowly clears
Connections:
- net SetSpeed_Analog renamed Analog
- net SetSpeed_PWM renamed PWM
Changed lines of the file:
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@@
     (effects (font (size 1.27 1.27)) (justify left bottom))
+  )
+  (hierarchical_label "Analog" (shape output) (at 209.55 83.82 0)
+    (effects (font (size 1.27 1.27)) (justify left))
+  )
+  (hierarchical_label "PWM" (shape input) (at 96.52 81.28 180)
+    (effects (font (size 1.27 1.27)) (justify right))
   )
   (symbol (lib_id "power:GND") (at 158.75 92.71 0) (unit 1)
