File: schematics/project/propshield.kicad_sch (KiCad schematic)
At the start: 1 part

Commit message: First steps with kicad structure -> kinda sucks
Parts:
- gave numbers to parts that had none: 1
Connections:
- net GND: now reaches U2.1 (GND)
- net GND: now also U2.10 (GND), U2.11 (GND), U2.12 (GND), U2.16 (GND), U2.17 (GND), U2.18 (GND), U2.19 (GND), U2.2 (GND), U2.22 (GND), U2.23 (GND), U2.24 (GND), U2.25 (GND), U2.29 (GND), U2.3 (GND), U2.31 (GND), U2.32 (GND), U2.37 (GND), U2.38 (GND), U2.5 (GND), U2.6 (GND)
- net MISO: now reaches U2.13 (MISO)
- net MOSI: now reaches U2.14 (MOSI)
- net SCK: now reaches U2.15 (SCK)
- net SDA: now reaches U2.20 (SDA)
- net SCL: now reaches U2.21 (SCL)
- net +3V3: now reaches U2.26 (3Vpower)
- net +3V3: now also U2.30 (3Vpower)
- net +5V: now reaches U2.28 (5VPower)
- net IRQ: now reaches U2.4 (IRQ)
- net CS: now reaches U2.8 (CS)
Other:
- moved on the sheet: U2

Commit message: small progress, angsthasen
Connections:
- net AGND: now reaches U2.27 (AGND)
- net AudioIN: now reaches U2.33 (AudioIN)
- net Speaker+: now reaches U2.39 (Speaker+)
- net Speaker-: now reaches U2.40 (Speaker-)
- net 5V_Speaker: now reaches U2.41 (5VPower)
- net AMP_EN: now reaches U2.7 (AMP_EN)
Changed lines of the file:
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@@
   (bus_alias "I2C_Motion" (members "SDA" "SCL" "IRQ"))
   (bus_alias "SPI_PS" (members "CS" "MISO" "MOSI" "SCK"))
+  (bus_alias "Speaker" (members "Speaker+" "Speaker-" "AMP_EN" "5V_Speaker" "AGND" "AudioIN"))
   (junction (at 72.39 95.25) (diameter 0) (color 0 0 0 0)
   )
@@
   (junction (at 72.39 110.49) (diameter 0) (color 0 0 0 0)
   )
+  (bus_entry (at 116.84 121.92) (size -2.54 2.54)
+    (stroke (width 0) (type default) (color 0 0 0 0))
+  )
   (bus_entry (at 113.03 91.44) (size 2.54 -2.54)
     (stroke (width 0) (type default) (color 0 0 0 0))
@@
     (stroke (width 0) (type default) (color 0 0 0 0))
   )
+  (bus_entry (at 116.84 116.84) (size -2.54 2.54)
+    (stroke (width 0) (type default) (color 0 0 0 0))
+  )
+  (bus_entry (at 116.84 109.22) (size -2.54 2.54)
+    (stroke (width 0) (type default) (color 0 0 0 0))
+  )
+  (bus_entry (at 116.84 119.38) (size -2.54 2.54)
+    (stroke (width 0) (type default) (color 0 0 0 0))
+  )
   (bus_entry (at 113.03 82.55) (size 2.54 -2.54)
     (stroke (width 0) (type default) (color 0 0 0 0))
@@
     (stroke (width 0) (type default) (color 0 0 0 0))
   )
+  (bus_entry (at 116.84 111.76) (size -2.54 2.54)
+    (stroke (width 0) (type default) (color 0 0 0 0))
+  )
+  (bus_entry (at 116.84 114.3) (size -2.54 2.54)
+    (stroke (width 0) (type default) (color 0 0 0 0))
+  )
   (wire (pts (xy 100.33 91.44) (xy 113.03 91.44))
     (stroke (width 0) (type default) (color 0 0 0 0))
   )
+  (bus (pts (xy 116.84 119.38) (xy 116.84 121.92))
+    (stroke (width 0) (type default) (color 0 0 0 0))
+  )
   (wire (pts (xy 74.93 110.49) (xy 72.39 110.49))
     (stroke (width 0) (type default) (color 0 0 0 0))
@@
     (stroke (width 0) (type default) (color 0 0 0 0))
   )
+  (wire (pts (xy 100.33 124.46) (xy 114.3 124.46))
+    (stroke (width 0) (type default) (color 0 0 0 0))
+  )
   (bus (pts (xy 115.57 83.82) (xy 115.57 86.36))
     (stroke (width 0) (type default) (color 0 0 0 0))
   )
+  (bus (pts (xy 116.84 109.22) (xy 116.84 111.76))
+    (stroke (width 0) (type default) (color 0 0 0 0))
+  )
+  (bus (pts (xy 116.84 111.76) (xy 116.84 114.3))
+    (stroke (width 0) (type default) (color 0 0 0 0))
+  )
   (wire (pts (xy 72.39 130.81) (xy 72.39 133.35))
     (stroke (width 0) (type default) (color 0 0 0 0))
@@
     (stroke (width 0) (type default) (color 0 0 0 0))
   )
+  (wire (pts (xy 100.33 116.84) (xy 114.3 116.84))
+    (stroke (width 0) (type default) (color 0 0 0 0))
+  )
   (bus (pts (xy 115.57 77.47) (xy 115.57 80.01))
     (stroke (width 0) (type default) (color 0 0 0 0))
@@
     (stroke (width 0) (type default) (color 0 0 0 0))
   )
+  (wire (pts (xy 100.33 114.3) (xy 114.3 114.3))
+    (stroke (width 0) (type default) (color 0 0 0 0))
+  )
   (wire (pts (xy 100.33 82.55) (xy 113.03 82.55))
     (stroke (width 0) (type default) (color 0 0 0 0))
@@
     (stroke (width 0) (type default) (color 0 0 0 0))
   )
+  (bus (pts (xy 116.84 114.3) (xy 116.84 116.84))
+    (stroke (width 0) (type default) (color 0 0 0 0))
+  )
   (wire (pts (xy 66.04 80.01) (xy 74.93 80.01))
     (stroke (width 0) (type default) (color 0 0 0 0))
@@
     (stroke (width 0) (type default) (color 0 0 0 0))
   )
+  (bus (pts (xy 116.84 116.84) (xy 116.84 119.38))
+    (stroke (width 0) (type default) (color 0 0 0 0))
+  )
   (wire (pts (xy 72.39 125.73) (xy 72.39 128.27))
     (stroke (width 0) (type default) (color 0 0 0 0))
@@
     (stroke (width 0) (type default) (color 0 0 0 0))
   )
+  (wire (pts (xy 100.33 111.76) (xy 114.3 111.76))
+    (stroke (width 0) (type default) (color 0 0 0 0))
+  )
   (wire (pts (xy 72.39 87.63) (xy 72.39 90.17))
     (stroke (width 0) (type default) (color 0 0 0 0))
@@
     (stroke (width 0) (type default) (color 0 0 0 0))
   )
+  (wire (pts (xy 100.33 121.92) (xy 114.3 121.92))
+    (stroke (width 0) (type default) (color 0 0 0 0))
+  )
   (wire (pts (xy 72.39 92.71) (xy 74.93 92.71))
     (stroke (width 0) (type default) (color 0 0 0 0))
@@
     (stroke (width 0) (type default) (color 0 0 0 0))
   )
+  (bus (pts (xy 130.81 109.22) (xy 116.84 109.22))
+    (stroke (width 0) (type default) (color 0 0 0 0))
+  )
   (bus (pts (xy 115.57 83.82) (xy 139.7 83.82))
+    (stroke (width 0) (type default) (color 0 0 0 0))
+  )
+  (wire (pts (xy 100.33 119.38) (xy 114.3 119.38))
     (stroke (width 0) (type default) (color 0 0 0 0))
   )
@@
     (effects (font (size 1.27 1.27)) (justify left bottom))
   )
-  (label "SDA" (at 104.14 80.01 0)
-    (effects (font (size 1.27 1.27)) (justify left bottom))
-  )
-  (label "MISO" (at 104.14 88.9 0)
+  (label "AGND" (at 102.87 124.46 0)
+    (effects (font (size 1.27 1.27)) (justify left bottom))
+  )
+  (label "SDA" (at 102.87 80.01 0)
+    (effects (font (size 1.27 1.27)) (justify left bottom))
+  )
+  (label "MISO" (at 102.87 88.9 0)
     (effects (font (size 1.27 1.27)) (justify left bottom))
   )
@@
     (effects (font (size 1.27 1.27)) (justify left bottom))
   )
-  (label "IRQ" (at 104.14 77.47 0)
-    (effects (font (size 1.27 1.27)) (justify left bottom))
-  )
-  (label "CS" (at 104.14 86.36 0)
-    (effects (font (size 1.27 1.27)) (justify left bottom))
-  )
-  (label "SCL" (at 104.14 82.55 0)
-    (effects (font (size 1.27 1.27)) (justify left bottom))
-  )
-  (label "MOSI" (at 104.14 91.44 0)
-    (effects (font (size 1.27 1.27)) (justify left bottom))
-  )
-  (label "SCK" (at 104.14 93.98 0)
-    (effects (font (size 1.27 1.27)) (justify left bottom))
+  (label "AMP_EN" (at 102.87 119.38 0)
+    (effects (font (size 1.27 1.27)) (justify left bottom))
+  )
+  (label "{Speaker" (at 120.65 109.22 0)
+    (effects (font (size 1.27 1.27)) (justify left bottom))
+  )
+  (label "5V_Speaker" (at 102.87 116.84 0)
+    (effects (font (size 1.27 1.27)) (justify left bottom))
+  )
+  (label "IRQ" (at 102.87 77.47 0)
+    (effects (font (size 1.27 1.27)) (justify left bottom))
+  )
+  (label "CS" (at 102.87 86.36 0)
+    (effects (font (size 1.27 1.27)) (justify left bottom))
+  )
+  (label "SCL" (at 102.87 82.55 0)
+    (effects (font (size 1.27 1.27)) (justify left bottom))
+  )
+  (label "MOSI" (at 102.87 91.44 0)
+    (effects (font (size 1.27 1.27)) (justify left bottom))
+  )
+  (label "Speaker-" (at 102.87 114.3 0)
+    (effects (font (size 1.27 1.27)) (justify left bottom))
+  )
+  (label "AudioIN" (at 102.87 121.92 0)
+    (effects (font (size 1.27 1.27)) (justify left bottom))
+  )
+  (label "SCK" (at 102.87 93.98 0)
+    (effects (font (size 1.27 1.27)) (justify left bottom))
+  )
+  (label "Speaker+" (at 102.87 111.76 0)
+    (effects (font (size 1.27 1.27)) (justify left bottom))
+  )
+  (hierarchical_label "Speaker" (shape output) (at 130.81 109.22 0)
+    (effects (font (size 1.27 1.27)) (justify left))
   )
   (hierarchical_label "{SPI_PS}" (shape bidirectional) (at 139.7 83.82 0)

Commit message: Adding separate library, BT Module
Parts:
- added C10, C8: 100nF 10V, Capacitor_SMD:C_0603_1608Metric, symbol Device:C
- added C11, C9: 1uF 10V, Capacitor_SMD:C_0603_1608Metric, symbol Device:C
Connections:
- net +3V3: now also C10.1, C11.1
- net +5V: now also C8.1, C9.1
- net GND: now also C10.2, C11.2, C8.2, C9.2
Changed lines of the file:
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@@
+    (stroke (width 0) (type default) (color 0 0 0 0))
+  )
+  (wire (pts (xy 162.56 82.55) (xy 162.56 85.09))
     (stroke (width 0) (type default) (color 0 0 0 0))
   )
@@
     (stroke (width 0) (type default) (color 0 0 0 0))
   )
+  (wire (pts (xy 27.94 68.58) (xy 27.94 71.12))
+    (stroke (width 0) (type default) (color 0 0 0 0))
+  )
   (wire (pts (xy 72.39 113.03) (xy 74.93 113.03))
     (stroke (width 0) (type default) (color 0 0 0 0))
@@
     (stroke (width 0) (type default) (color 0 0 0 0))
   )
+  (wire (pts (xy 45.72 78.74) (xy 45.72 81.28))
+    (stroke (width 0) (type default) (color 0 0 0 0))
+  )
+  (wire (pts (xy 180.34 72.39) (xy 180.34 74.93))
+    (stroke (width 0) (type default) (color 0 0 0 0))
+  )
   (wire (pts (xy 66.04 80.01) (xy 74.93 80.01))
     (stroke (width 0) (type default) (color 0 0 0 0))
   )
+  (wire (pts (xy 27.94 78.74) (xy 27.94 81.28))
+    (stroke (width 0) (type default) (color 0 0 0 0))
+  )
   (wire (pts (xy 74.93 77.47) (xy 72.39 77.47))
     (stroke (width 0) (type default) (color 0 0 0 0))
@@
     (stroke (width 0) (type default) (color 0 0 0 0))
   )
+  (wire (pts (xy 180.34 82.55) (xy 180.34 85.09))
+    (stroke (width 0) (type default) (color 0 0 0 0))
+  )
   (wire (pts (xy 72.39 125.73) (xy 72.39 128.27))
     (stroke (width 0) (type default) (color 0 0 0 0))
@@
     (stroke (width 0) (type default) (color 0 0 0 0))
   )
+  (wire (pts (xy 45.72 68.58) (xy 45.72 71.12))
+    (stroke (width 0) (type default) (color 0 0 0 0))
+  )
   (wire (pts (xy 100.33 121.92) (xy 114.3 121.92))
     (stroke (width 0) (type default) (color 0 0 0 0))
@@
   )
   (wire (pts (xy 72.39 85.09) (xy 72.39 87.63))
+    (stroke (width 0) (type default) (color 0 0 0 0))
+  )
+  (wire (pts (xy 162.56 72.39) (xy 162.56 74.93))
     (stroke (width 0) (type default) (color 0 0 0 0))
   )
@@
   (hierarchical_label "{I2C_Motion}" (shape bidirectional) (at 139.7 74.93 0)
     (effects (font (size 1.27 1.27)) (justify left))
+  )
+  (symbol (lib_id "power:+5V") (at 27.94 68.58 0) (unit 1)
+    (in_bom yes) (on_board yes) (fields_autoplaced)
+    (property "Reference" "#PWR09" (id 0) (at 27.94 72.39 0)
+      (effects (font (size 1.27 1.27)) hide)
+    )
+    (property "Value" "+5V" (id 1) (at 27.94 63.5 0))
+    (property "Footprint" "" (id 2) (at 27.94 68.58 0)
+      (effects (font (size 1.27 1.27)) hide)
+    )
+    (property "Datasheet" "" (id 3) (at 27.94 68.58 0)
+      (effects (font (size 1.27 1.27)) hide)
+    )
+    (pin "1")
   )
   (symbol (lib_name "PropShieldMotionSens_1") (lib_id "IceWheelLib:PropShieldMotionSens") (at 100.33 77.47 0) (mirror y) (unit 1)
@@
     (pin "9")
   )
+  (symbol (lib_id "power:+5V") (at 45.72 68.58 0) (unit 1)
+    (in_bom yes) (on_board yes) (fields_autoplaced)
+    (property "Reference" "#PWR011" (id 0) (at 45.72 72.39 0)
+      (effects (font (size 1.27 1.27)) hide)
+    )
+    (property "Value" "+5V" (id 1) (at 45.72 63.5 0))
+    (property "Footprint" "" (id 2) (at 45.72 68.58 0)
+      (effects (font (size 1.27 1.27)) hide)
+    )
+    (property "Datasheet" "" (id 3) (at 45.72 68.58 0)
+      (effects (font (size 1.27 1.27)) hide)
+    )
+    (pin "1")
+  )
   (symbol (lib_id "power:+5V") (at 72.39 74.93 0) (unit 1)
     (in_bom yes) (on_board yes) (fields_autoplaced)
@@
     (pin "1")
   )
+  (symbol (lib_id "power:+3V3") (at 180.34 72.39 0) (unit 1)
+    (in_bom yes) (on_board yes) (fields_autoplaced)
+    (property "Reference" "#PWR015" (id 0) (at 180.34 76.2 0)
+      (effects (font (size 1.27 1.27)) hide)
+    )
+    (property "Value" "+3V3" (id 1) (at 180.34 67.31 0))
+    (property "Footprint" "" (id 2) (at 180.34 72.39 0)
+      (effects (font (size 1.27 1.27)) hide)
+    )
+    (property "Datasheet" "" (id 3) (at 180.34 72.39 0)
+      (effects (font (size 1.27 1.27)) hide)
+    )
+    (pin "1")
+  )
+  (symbol (lib_id "Device:C") (at 27.94 74.93 0) (unit 1)
+    (in_bom no) (on_board yes) (fields_autoplaced)
+    (property "Reference" "C8" (id 0) (at 31.75 73.6599 0)
+      (effects (font (size 1.27 1.27)) (justify left))
+    )
+    (property "Value" "100nF 10V" (id 1) (at 31.75 76.1999 0)
+      (effects (font (size 1.27 1.27)) (justify left))
+    )
+    (property "Footprint" "Capacitor_SMD:C_0603_1608Metric" (id 2) (at 28.9052 78.74 0)
+      (effects (font (size 1.27 1.27)) hide)
+    )
+    (property "Datasheet" "~" (id 3) (at 27.94 74.93 0)
+      (effects (font (size 1.27 1.27)) hide)
+    )
+    (pin "1")
+    (pin "2")
+  )
+  (symbol (lib_id "power:GND") (at 45.72 81.28 0) (unit 1)
+    (in_bom yes) (on_board yes) (fields_autoplaced)
+    (property "Reference" "#PWR012" (id 0) (at 45.72 87.63 0)
+      (effects (font (size 1.27 1.27)) hide)
+    )
+    (property "Value" "GND" (id 1) (at 45.72 86.36 0))
+    (property "Footprint" "" (id 2) (at 45.72 81.28 0)
+      (effects (font (size 1.27 1.27)) hide)
+    )
+    (property "Datasheet" "" (id 3) (at 45.72 81.28 0)
+      (effects (font (size 1.27 1.27)) hide)
+    )
+    (pin "1")
+  )
   (symbol (lib_id "power:+3V3") (at 66.04 74.93 0) (unit 1)
     (in_bom yes) (on_board yes) (fields_autoplaced)
@@
     (pin "1")
   )
+  (symbol (lib_id "power:GND") (at 162.56 85.09 0) (unit 1)
+    (in_bom yes) (on_board yes) (fields_autoplaced)
+    (property "Reference" "#PWR014" (id 0) (at 162.56 91.44 0)
+      (effects (font (size 1.27 1.27)) hide)
+    )
+    (property "Value" "GND" (id 1) (at 162.56 90.17 0))
+    (property "Footprint" "" (id 2) (at 162.56 85.09 0)
+      (effects (font (size 1.27 1.27)) hide)
+    )
+    (property "Datasheet" "" (id 3) (at 162.56 85.09 0)
+      (effects (font (size 1.27 1.27)) hide)
+    )
+    (pin "1")
+  )
+  (symbol (lib_id "Device:C") (at 162.56 78.74 0) (unit 1)
+    (in_bom no) (on_board yes) (fields_autoplaced)
+    (property "Reference" "C10" (id 0) (at 166.37 77.4699 0)
+      (effects (font (size 1.27 1.27)) (justify left))
+    )
+    (property "Value" "100nF 10V" (id 1) (at 166.37 80.0099 0)
+      (effects (font (size 1.27 1.27)) (justify left))
+    )
+    (property "Footprint" "Capacitor_SMD:C_0603_1608Metric" (id 2) (at 163.5252 82.55 0)
+      (effects (font (size 1.27 1.27)) hide)
+    )
+    (property "Datasheet" "~" (id 3) (at 162.56 78.74 0)
+      (effects (font (size 1.27 1.27)) hide)
+    )
+    (pin "1")
+    (pin "2")
+  )
+  (symbol (lib_id "power:GND") (at 27.94 81.28 0) (unit 1)
+    (in_bom yes) (on_board yes) (fields_autoplaced)
+    (property "Reference" "#PWR010" (id 0) (at 27.94 87.63 0)
+      (effects (font (size 1.27 1.27)) hide)
+    )
+    (property "Value" "GND" (id 1) (at 27.94 86.36 0))
+    (property "Footprint" "" (id 2) (at 27.94 81.28 0)
+      (effects (font (size 1.27 1.27)) hide)
+    )
+    (property "Datasheet" "" (id 3) (at 27.94 81.28 0)
+      (effects (font (size 1.27 1.27)) hide)
+    )
+    (pin "1")
+  )
+  (symbol (lib_id "power:+3V3") (at 162.56 72.39 0) (unit 1)
+    (in_bom yes) (on_board yes) (fields_autoplaced)
+    (property "Reference" "#PWR013" (id 0) (at 162.56 76.2 0)
+      (effects (font (size 1.27 1.27)) hide)
+    )
+    (property "Value" "+3V3" (id 1) (at 162.56 67.31 0))
+    (property "Footprint" "" (id 2) (at 162.56 72.39 0)
+      (effects (font (size 1.27 1.27)) hide)
+    )
+    (property "Datasheet" "" (id 3) (at 162.56 72.39 0)
+      (effects (font (size 1.27 1.27)) hide)
+    )
+    (pin "1")
+  )
+  (symbol (lib_id "power:GND") (at 180.34 85.09 0) (unit 1)
+    (in_bom yes) (on_board yes) (fields_autoplaced)
+    (property "Reference" "#PWR016" (id 0) (at 180.34 91.44 0)
+      (effects (font (size 1.27 1.27)) hide)
+    )
+    (property "Value" "GND" (id 1) (at 180.34 90.17 0))
+    (property "Footprint" "" (id 2) (at 180.34 85.09 0)
+      (effects (font (size 1.27 1.27)) hide)
+    )
+    (property "Datasheet" "" (id 3) (at 180.34 85.09 0)
+      (effects (font (size 1.27 1.27)) hide)
+    )
+    (pin "1")
+  )
+  (symbol (lib_id "Device:C") (at 180.34 78.74 0) (unit 1)
+    (in_bom no) (on_board yes) (fields_autoplaced)
+    (property "Reference" "C11" (id 0) (at 184.15 77.4699 0)
+      (effects (font (size 1.27 1.27)) (justify left))
+    )
+    (property "Value" "1uF 10V" (id 1) (at 184.15 80.0099 0)
+      (effects (font (size 1.27 1.27)) (justify left))
+    )
+    (property "Footprint" "Capacitor_SMD:C_0603_1608Metric" (id 2) (at 181.3052 82.55 0)
+      (effects (font (size 1.27 1.27)) hide)
+    )
+    (property "Datasheet" "~" (id 3) (at 180.34 78.74 0)
+      (effects (font (size 1.27 1.27)) hide)
+    )
+    (pin "1")
+    (pin "2")
+  )
   (symbol (lib_id "power:GND") (at 72.39 138.43 0) (unit 1)
     (in_bom yes) (on_board yes) (fields_autoplaced)
@@
     (pin "1")
   )
+  (symbol (lib_id "Device:C") (at 45.72 74.93 0) (unit 1)
+    (in_bom no) (on_board yes) (fields_autoplaced)
+    (property "Reference" "C9" (id 0) (at 49.53 73.6599 0)
+      (effects (font (size 1.27 1.27)) (justify left))
+    )
+    (property "Value" "1uF 10V" (id 1) (at 49.53 76.1999 0)
+      (effects (font (size 1.27 1.27)) (justify left))
+    )
+    (property "Footprint" "Capacitor_SMD:C_0603_1608Metric" (id 2) (at 46.6852 78.74 0)
+      (effects (font (size 1.27 1.27)) hide)
+    )
+    (property "Datasheet" "~" (id 3) (at 45.72 74.93 0)
+      (effects (font (size 1.27 1.27)) hide)
+    )
+    (pin "1")
+    (pin "2")
+  )
 )

Commit message: random commit
Other:
- note added: "- Motion sensors - spi to teensy - LED driver - Audio Steckerleiste separat anlöten"
- note removed: "-Motion sensors -spi to teensy - LED driver - Audio"
- moved on the sheet: C10, C11, U2
